File: pce-gt-controller.kicad_sch (KiCad schematic)
At the start: 30 parts, among them CN800 Conn_01x12, CN801 AUDIO, J800 LINK, SW801 I, SW802 II, SW803 SELECT, SW804 RUN, SW805 UP, SW806 RIGHT, SW807 DOWN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

Commit message: Update pce-gt-controller.kicad_sch
Parts:
- CC800: value 47nF -> 47uF 6.3v
Changed lines of the file:
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@@
   (symbol (lib_id "Device:C_Small") (at 146.685 172.72 90) (unit 1)
     (in_bom yes) (on_board yes) (dnp no)
-    (property "Reference" "C800" (at 149.225 167.64 90)
-      (effects (font (size 1.27 1.27)) (justify left))
-    )
-    (property "Value" "10nF" (at 149.225 170.18 90)
+    (property "Reference" "C800" (at 159.385 170.815 90)
+      (effects (font (size 1.27 1.27)) (justify left))
+    )
+    (property "Value" "10nF" (at 159.385 172.72 90)
       (effects (font (size 1.27 1.27)) (justify left))
     )
@@
   (symbol (lib_id "Device:C_Polarized_Small") (at 146.685 177.8 90) (mirror x) (unit 1)
     (in_bom yes) (on_board yes) (dnp no)
-    (property "Reference" "CC800" (at 146.685 180.34 90)
-      (effects (font (size 1.27 1.27)))
-    )
-    (property "Value" "47nF" (at 146.685 182.88 90)
-      (effects (font (size 1.27 1.27)))
-    )
+    (property "Reference" "CC800" (at 156.845 177.8 90)
+      (effects (font (size 1.27 1.27)))
+    )
+    (property "Value" "47uF 6.3v" (at 156.845 179.705 90)
+      (effects (font (size 1.27 1.27)))
+    )

Commit message: Update pce-gt-controller.kicad_sch
Parts:
- C801: value 10nF -> 15nF
Changed lines of the file:
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@@
   (symbol (lib_id "Device:R_Small") (at 115.57 82.55 90) (unit 1)
     (in_bom yes) (on_board yes) (dnp no)
-    (property "Reference" "R800" (at 118.11 72.39 90)
-      (effects (font (size 1.27 1.27)) (justify left))
-    )
-    (property "Value" "R_Small" (at 127 72.39 90)
+    (property "Reference" "R800" (at 102.87 82.55 90)
+      (effects (font (size 1.27 1.27)) (justify left))
+    )
+    (property "Value" "R_Small" (at 111.76 82.55 90)
       (effects (font (size 1.27 1.27)) (justify left))
     )
@@
   (symbol (lib_id "Device:C_Small") (at 115.57 87.63 270) (unit 1)
     (in_bom yes) (on_board yes) (dnp no)
-    (property "Reference" "C801" (at 118.11 76.1936 90)
+    (property "Reference" "C801" (at 102.87 87.63 90)
       (effects (font (size 1.27 1.27)) (justify right))
     )
-    (property "Value" "10nF" (at 124.46 76.2 90)
+    (property "Value" "15nF" (at 111.76 87.63 90)
       (effects (font (size 1.27 1.27)) (justify right))
     )
@@
   (symbol (lib_id "Device:R_Small") (at 115.57 85.09 90) (unit 1)
     (in_bom yes) (on_board yes) (dnp no)
-    (property "Reference" "R801" (at 118.11 74.295 90)
-      (effects (font (size 1.27 1.27)) (justify left))
-    )
-    (property "Value" "R_Small" (at 127 74.295 90)
-      (effects (font (size 1.27 1.27)) (justify left))
-    )
+    (property "Reference" "R801" (at 102.87 85.09 90)
+      (effects (font (size 1.27 1.27)) (justify left))
+    )
+    (property "Value" "R_Small" (at 111.76 85.09 90)
+      (effects (font (size 1.27 1.27)) (justify left))
+    )
