File: pce-gt-controller.kicad_sch (KiCad schematic)
At the start: 30 parts, among them CN800 Conn_01x12, CN801 AUDIO, J800 LINK, SW801 I, SW802 II, SW803 SELECT, SW804 RUN, SW805 UP, SW806 RIGHT, SW807 DOWN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

Commit message: Updates
Parts:
- C800, C801, L803, L804, L805, R800, R801, R803, R804: footprint (none) -> GT Controller:Resistor 0805 SMD
- D800, D801, D802: footprint Package_TO_SOT_SMD:SOT-23 -> GT Controller:Diode SOT-23
- L800, L801, L802: footprint (none) -> GT Controller:Ferrite
- UIC800: footprint (none) -> GT Controller:IC800
Changed lines of the file:
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@@
       (effects (font (size 1.27 1.27)))
     )
-    (property "Footprint" "Package_TO_SOT_SMD:SOT-23" (at 230.505 59.69 0)
+    (property "Footprint" "GT Controller:Diode SOT-23" (at 230.505 59.69 0)
       (effects (font (size 1.27 1.27)) hide)
     )
@@
       (effects (font (size 1.27 1.27)) (justify left) hide)
     )
-    (property "Footprint" "" (at 242.57 83.312 90)
+    (property "Footprint" "GT Controller:Resistor 0805 SMD" (at 242.57 83.312 90)
       (effects (font (size 1.27 1.27)) hide)
     )
@@
       (effects (font (size 1.27 1.27)) (justify left) hide)
     )
-    (property "Footprint" "" (at 249.555 83.312 90)
+    (property "Footprint" "GT Controller:Ferrite" (at 249.555 83.312 90)
       (effects (font (size 1.27 1.27)) hide)
     )
@@
       (effects (font (size 1.27 1.27)) (justify left))
     )
-    (property "Footprint" "" (at 146.05 73.66 0)
+    (property "Footprint" "GT Controller:IC800" (at 146.05 73.66 0)
       (effects (font (size 1.27 1.27)) hide)
     )
@@
       (effects (font (size 1.27 1.27)))
     )
-    (property "Footprint" "Package_TO_SOT_SMD:SOT-23" (at 230.505 83.185 0)
+    (property "Footprint" "GT Controller:Diode SOT-23" (at 230.505 83.185 0)
       (effects (font (size 1.27 1.27)) hide)
     )
@@
       (effects (font (size 1.27 1.27)) (justify left))
     )
-    (property "Footprint" "" (at 238.125 80.645 0)
+    (property "Footprint" "GT Controller:Resistor 0805 SMD" (at 238.125 80.645 0)
       (effects (font (size 1.27 1.27)) hide)
     )
@@
       (effects (font (size 1.27 1.27)) (justify left))
     )
-    (property "Footprint" "" (at 115.57 82.55 0)
+    (property "Footprint" "GT Controller:Resistor 0805 SMD" (at 115.57 82.55 0)
       (effects (font (size 1.27 1.27)) hide)
     )
@@
       (effects (font (size 1.27 1.27)) (justify left))
     )
-    (property "Footprint" "Package_TO_SOT_SMD:SOT-23" (at 135.255 175.26 0)
+    (property "Footprint" "GT Controller:Diode SOT-23" (at 135.255 175.26 0)
       (effects (font (size 1.27 1.27)) hide)
     )
@@
       (effects (font (size 1.27 1.27)) (justify right))
     )
-    (property "Footprint" "" (at 115.57 87.63 0)
+    (property "Footprint" "GT Controller:Resistor 0805 SMD" (at 115.57 87.63 0)
       (effects (font (size 1.27 1.27)) hide)
     )
@@
       (effects (font (size 1.27 1.27)) (justify left) hide)
     )
-    (property "Footprint" "" (at 249.555 99.187 90)
+    (property "Footprint" "GT Controller:Ferrite" (at 249.555 99.187 90)
       (effects (font (size 1.27 1.27)) hide)
     )
@@
       (effects (font (size 1.27 1.27)) (justify left))
     )
-    (property "Footprint" "" (at 238.125 57.15 0)
+    (property "Footprint" "GT Controller:Resistor 0805 SMD" (at 238.125 57.15 0)
       (effects (font (size 1.27 1.27)) hide)
     )
@@
       (effects (font (size 1.27 1.27)) (justify left))
     )
-    (property "Footprint" "" (at 146.685 172.72 0)
+    (property "Footprint" "GT Controller:Resistor 0805 SMD" (at 146.685 172.72 0)
       (effects (font (size 1.27 1.27)) hide)
     )
@@
       (effects (font (size 1.27 1.27)) (justify left) hide)
     )
-    (property "Footprint" "" (at 249.555 59.817 90)
+    (property "Footprint" "GT Controller:Ferrite" (at 249.555 59.817 90)
       (effects (font (size 1.27 1.27)) hide)
     )
@@
       (effects (font (size 1.27 1.27)) (justify left) hide)
     )
-    (property "Footprint" "" (at 242.57 99.187 90)
+    (property "Footprint" "GT Controller:Resistor 0805 SMD" (at 242.57 99.187 90)
       (effects (font (size 1.27 1.27)) hide)
     )
@@
       (effects (font (size 1.27 1.27)) (justify left))
     )
-    (property "Footprint" "" (at 115.57 85.09 0)
+    (property "Footprint" "GT Controller:Resistor 0805 SMD" (at 115.57 85.09 0)
       (effects (font (size 1.27 1.27)) hide)
     )
@@
       (effects (font (size 1.27 1.27)) (justify left) hide)
     )
-    (property "Footprint" "" (at 242.57 59.817 90)
-      (effects (font (size 1.27 1.27)) hide)
-    )
+    (property "Footprint" "GT Controller:Resistor 0805 SMD" (at 242.57 59.817 90)
+      (effects (font (size 1.27 1.27)) hide)
+    )

Commit message: Updates
Parts:
- CC800: footprint (none) -> GT Controller:CC800 Electrolytic
- CN800: footprint (none) -> GT Controller:CN800
- SW801: footprint (none) -> GT Controller:Switch Type 3
- SW802: footprint (none) -> GT Controller:Switch Type 2
- SW803, SW804: footprint (none) -> GT Controller:Switch Type 1
- SW805: footprint (none) -> Connector_PinHeader_1.00mm:PinHeader_1x02_P1.00mm_Vertical
- SW806, SW808: footprint (none) -> GT Controller:Switch Type 5
- SW807: footprint (none) -> GT Controller:Switch Type 4
- renumbered UIC800 to IC800
Changed lines of the file:
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@@
   (symbol (lib_id "PCE:BU5782K") (at 146.05 73.66 0) (unit 1)
     (in_bom yes) (on_board yes) (dnp no) (fields_autoplaced)
-    (property "Reference" "UIC800" (at 148.2441 38.1 0)
+    (property "Reference" "IC800" (at 148.2441 38.1 0)
       (effects (font (size 1.27 1.27)) (justify left))
     )
@@
       (project "pce-gt-controller"
         (path "/56793d7b-9d4c-4af4-8ca8-6f6e67f49f0d"
-          (reference "UIC800") (unit 1)
+          (reference "IC800") (unit 1)
         )
       )
@@
       (effects (font (size 1.27 1.27)))
     )
-    (property "Footprint" "" (at 35.56 165.735 0)
+    (property "Footprint" "GT Controller:Switch Type 3" (at 35.56 165.735 0)
       (effects (font (size 1.27 1.27)) hide)
     )
@@
       (effects (font (size 1.27 1.27)))
     )
-    (property "Footprint" "" (at 35.56 128.905 0)
+    (property "Footprint" "GT Controller:Switch Type 1" (at 35.56 128.905 0)
       (effects (font (size 1.27 1.27)) hide)
     )
@@
       (effects (font (size 1.27 1.27)))
     )
-    (property "Footprint" "" (at 35.56 112.395 0)
+    (property "Footprint" "GT Controller:Switch Type 5" (at 35.56 112.395 0)
       (effects (font (size 1.27 1.27)) hide)
     )
@@
       (effects (font (size 1.27 1.27)))
     )
-    (property "Footprint" "" (at 35.56 137.16 0)
+    (property "Footprint" "GT Controller:Switch Type 1" (at 35.56 137.16 0)
       (effects (font (size 1.27 1.27)) hide)
     )
@@
       (effects (font (size 1.27 1.27)))
     )
-    (property "Footprint" "" (at 35.56 95.885 0)
+    (property "Footprint" "Connector_PinHeader_1.00mm:PinHeader_1x02_P1.00mm_Vertical" (at 35.56 95.885 0)
       (effects (font (size 1.27 1.27)) hide)
     )
@@
       (effects (font (size 1.27 1.27)))
     )
-    (property "Footprint" "" (at 35.56 180.975 0)
+    (property "Footprint" "GT Controller:Switch Type 2" (at 35.56 180.975 0)
       (effects (font (size 1.27 1.27)) hide)
     )
@@
       (effects (font (size 1.27 1.27)) hide)
     )
-    (property "Footprint" "" (at 20.32 33.02 0)
+    (property "Footprint" "GT Controller:CN800" (at 20.32 33.02 0)
       (effects (font (size 1.27 1.27)) hide)
     )
@@
       (effects (font (size 1.27 1.27)))
     )
-    (property "Footprint" "" (at 146.685 177.8 0)
+    (property "Footprint" "GT Controller:CC800 Electrolytic" (at 146.685 177.8 0)
       (effects (font (size 1.27 1.27)) hide)
     )
@@
       (effects (font (size 1.27 1.27)))
     )
-    (property "Footprint" "" (at 35.56 104.14 0)
+    (property "Footprint" "GT Controller:Switch Type 4" (at 35.56 104.14 0)
       (effects (font (size 1.27 1.27)) hide)
     )
@@
       (effects (font (size 1.27 1.27)))
     )
-    (property "Footprint" "" (at 35.56 120.65 0)
-      (effects (font (size 1.27 1.27)) hide)
-    )
+    (property "Footprint" "GT Controller:Switch Type 5" (at 35.56 120.65 0)
+      (effects (font (size 1.27 1.27)) hide)
+    )

Commit message: Fix Link
Connections:
- net LINK 1: now also D801.1 (A), D801.2 (A), L805.1, R803.2
- net LINK 2: now also D802.1 (A), D802.2 (A), L804.1, R804.2
Changed lines of the file:
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@@
   (junction (at 40.64 133.985) (diameter 0) (color 0 0 0 0)
   )
+  (junction (at 222.885 85.09) (diameter 0) (color 0 0 0 0)
+  )
   (junction (at 163.83 105.41) (diameter 0) (color 0 0 0 0)
   )
@@
   (junction (at 113.03 100.33) (diameter 0) (color 0 0 0 0)
   )
+  (junction (at 222.885 61.595) (diameter 0) (color 0 0 0 0)
+  )
   (junction (at 118.11 87.63) (diameter 0) (color 0 0 0 0)
   )
@@
     (stroke (width 0) (type default))
   )
+  (wire (pts (xy 219.71 61.595) (xy 222.885 61.595))
+    (stroke (width 0) (type default))
+  )
   (wire (pts (xy 66.04 183.515) (xy 57.785 183.515))
     (stroke (width 0) (type default))
@@
     (stroke (width 0) (type default))
   )
+  (wire (pts (xy 219.71 85.09) (xy 222.885 85.09))
+    (stroke (width 0) (type default))
+  )
   (wire (pts (xy 142.875 172.72) (xy 144.145 172.72))
     (stroke (width 0) (type default))
@@
     )
   )
+  (global_label "LINK 1" (shape input) (at 219.71 61.595 180) (fields_autoplaced)
+    (effects (font (size 1.27 1.27)) (justify right))
+    (property "Intersheetrefs" "${INTERSHEET_REFS}" (at 210.3143 61.595 0)
+      (effects (font (size 1.27 1.27)) (justify right) hide)
+    )
+  )
   (global_label "D0" (shape input) (at 43.18 22.86 0) (fields_autoplaced)
     (effects (font (size 1.27 1.27)) (justify left))
@@
     )
   )
+  (global_label "LINK 2" (shape input) (at 219.71 85.09 180) (fields_autoplaced)
+    (effects (font (size 1.27 1.27)) (justify right))
+    (property "Intersheetrefs" "${INTERSHEET_REFS}" (at 210.3143 85.09 0)
+      (effects (font (size 1.27 1.27)) (justify right) hide)
+    )
+  )

Commit message: Updates
Complete?
Parts:
- CN801: footprint (none) -> GT Controller:CN801
- J800: footprint (none) -> GT Controller:J800
- SW805: footprint Connector_PinHeader_1.00mm:PinHeader_1x02_P1.00mm_Vertical -> GT Controller:Switch Type 4
- SW809, SW810: footprint (none) -> GT Controller:Turbo Switch
Changed lines of the file:
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@@
       (effects (font (size 1.27 1.27)))
     )
-    (property "Footprint" "Connector_PinHeader_1.00mm:PinHeader_1x02_P1.00mm_Vertical" (at 35.56 95.885 0)
+    (property "Footprint" "GT Controller:Switch Type 4" (at 35.56 95.885 0)
       (effects (font (size 1.27 1.27)) hide)
     )
@@
       (effects (font (size 1.27 1.27)))
     )
-    (property "Footprint" "" (at 20.32 64.135 0)
+    (property "Footprint" "GT Controller:CN801" (at 20.32 64.135 0)
       (effects (font (size 1.27 1.27)) hide)
     )
@@
       (effects (font (size 1.27 1.27)))
     )
-    (property "Footprint" "" (at 236.22 126.365 0)
+    (property "Footprint" "GT Controller:J800" (at 236.22 126.365 0)
       (effects (font (size 1.27 1.27)) hide)
     )
@@
       (effects (font (size 1.27 1.27)))
     )
-    (property "Footprint" "" (at 36.83 166.37 0)
+    (property "Footprint" "GT Controller:Turbo Switch" (at 36.83 166.37 0)
       (effects (font (size 1.27 1.27)) hide)
     )
@@
       (effects (font (size 1.27 1.27)))
     )
-    (property "Footprint" "" (at 36.83 181.61 0)
-      (effects (font (size 1.27 1.27)) hide)
-    )
+    (property "Footprint" "GT Controller:Turbo Switch" (at 36.83 181.61 0)
+      (effects (font (size 1.27 1.27)) hide)
+    )
