File: remaster/pce-gt-controller.kicad_pcb (KiCad board)
At the start: 2 copper layers, 94 x 79.1 mm, 36 parts, among them CN800 Conn_01x12, CN801 AUDIO, J800 LINK, SW801 I, SW802 II, SW803 SELECT, SW804 RUN, SW805 UP, SW806 RIGHT, SW807 DOWN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

Commit message: Added BoardFolk Silk, Tidy up
Parts:
- added G***: LOGO, GT Controller:BoardFolk, B.Cu at (121.3, 63.1)
Other:
- board text added: "Schematics: Chrissy (@chris_jh) PCB Layout: Rob Taylor (@PeepoUK), Chrissy (@chris_jh) Support: Simon Lock (@A3rgan) Steve Maddison (@cosam_the_great) Leo Oliveria (@leo__oliveira) Zaxour 阿宅, (@zaxour) Ian Cudlip (@grandoldian) Dennis van den Broek (@PointerFunction)"
- board text added: "The Board Folk Team 2023 PC Engine GT Controller PCB (Remaster) - BF1.1"
