File: remaster/pce-gt-controller.kicad_sch (KiCad schematic)
At the start: 36 parts, among them CN800 Conn_01x12, CN801 AUDIO, J800 LINK, SW801 I, SW802 II, SW803 SELECT, SW804 RUN, SW805 UP, SW806 RIGHT, SW807 DOWN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

Commit message: Added BoardFolk Silk, Tidy up
Other:
- company: (none) -> The Board Folk Team
- title: (none) -> PC Engine GT Controller PCB (Remaster)
Changed lines of the file:
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@@
 (kicad_sch (version 20230121) (generator eeschema)
   (paper "A4")
+  (title_block
+    (title "PC Engine GT Controller PCB (Remaster)")
+    (date "2023-12-31")
+    (rev "BF1.1")
+    (company "The Board Folk Team")
+  )
   (junction (at 142.24 57.15) (diameter 0) (color 0 0 0 0)
   )
